File: sheets/clock-input/clock-input.kicad_sch (KiCad schematic)
At the start: 5 parts, among them U1 40106

Commit message: Give the blocks a real interface
Interface nets on gate-output, cv-output and clock-input were plain net
labels. A plain label is scoped to its sheet and never becomes a sheet
pin, so a parent module could not reach any of them. They are now
hierarchical labels with input and output shapes.

power-input needed no change: its interface is the header and the global
rails, and its labels are internal to the sheet. regulator-5v has no
labels at all.

Two defects found while checking: power-input carried no footprints on
any part and clock-input carried none on U1, both from the Konnect drop.
Every block also had unannotated power flags. Fixed.

All six blocks: ERC 0 errors.

Co-Authored-By: Claude Opus 5 (1M context) <noreply@anthropic.com>
Parts:
- U1: footprint (none) -> Eurorack Common:DIP-14_W7.62mm
