File: sheets/power-input/power-input.kicad_sch (KiCad schematic)
At the start: 5 parts, among them J1 Eurorack Power

Commit message: Give the blocks a real interface
Interface nets on gate-output, cv-output and clock-input were plain net
labels. A plain label is scoped to its sheet and never becomes a sheet
pin, so a parent module could not reach any of them. They are now
hierarchical labels with input and output shapes.

power-input needed no change: its interface is the header and the global
rails, and its labels are internal to the sheet. regulator-5v has no
labels at all.

Two defects found while checking: power-input carried no footprints on
any part and clock-input carried none on U1, both from the Konnect drop.
Every block also had unannotated power flags. Fixed.

All six blocks: ERC 0 errors.

Co-Authored-By: Claude Opus 5 (1M context) <noreply@anthropic.com>
Parts:
- C1, C2: footprint (none) -> Eurorack Common:CP_Radial_D5.0mm_H11.0mm_P2.00mm
- D1, D2: footprint (none) -> Eurorack Common:D_DO-41_SOD81_P7.62mm_Horizontal
- J1: footprint (none) -> Eurorack Common:Eurorack Power Header (10 pin)
Changed lines of the file:
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@@
 			(project "power-input"
 				(path "/6f1c29c3-265e-4aa9-b46d-a6f87ca6134a"
-					(reference "?")
+					(reference "1")
 					(unit 1)
 				)
@@
 			(project "power-input"
 				(path "/6f1c29c3-265e-4aa9-b46d-a6f87ca6134a"
-					(reference "?")
+					(reference "2")
 					(unit 1)
 				)
@@
 			)
 		)
-		(property "Footprint" ""
+		(property "Footprint" "Eurorack Common:CP_Radial_D5.0mm_H11.0mm_P2.00mm"
 			(at 109.22 76.2 0)
 			(hide yes)
@@
 			)
 		)
-		(property "Footprint" ""
+		(property "Footprint" "Eurorack Common:CP_Radial_D5.0mm_H11.0mm_P2.00mm"
 			(at 109.22 101.6 0)
 			(hide yes)
@@
 			)
 		)
-		(property "Footprint" ""
+		(property "Footprint" "Eurorack Common:D_DO-41_SOD81_P7.62mm_Horizontal"
 			(at 88.9 76.2 0)
 			(hide yes)
@@
 			(project "power-input"
 				(path "/6f1c29c3-265e-4aa9-b46d-a6f87ca6134a"
-					(reference "?")
+					(reference "3")
 					(unit 1)
 				)
@@
 			)
 		)
-		(property "Footprint" ""
+		(property "Footprint" "Eurorack Common:D_DO-41_SOD81_P7.62mm_Horizontal"
 			(at 88.9 101.6 0)
 			(hide yes)
@@
 			)
 		)
-		(property "Footprint" ""
+		(property "Footprint" "Eurorack Common:Eurorack Power Header (10 pin)"
 			(at 40.64 88.9 0)
 			(hide yes)
